Commit message: trying dreal regions again

File: manipulation/models/planar_iiwa14_one_sphere.urdf (robot description, URDF)
Before this commit: robot iiwa14, 10 links, 9 joints
Links:
- link iiwa_link_7: geometry collision box size=.12 .12 .12; visual mesh filename=package://iiwa_description/meshes/visual/link_7.obj
