Commit message: fix for package.xml files removed from drake

File: manipulation/models/two_link_iiwa14.urdf (robot description, URDF)
Before this commit: robot iiwa14, 10 links, 9 joints
Links:
- link iiwa_link_0: geometry collision cylinder length=0.17 radius=0.139; visual mesh filename=package://drake/manipulation/models/iiwa_description/meshes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
- link iiwa_link_1: geometry collision sphere radius=0.07959901601; visual mesh filename=package://drake/manipulation/models/iiwa_description/meshes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
- link iiwa_link_2: geometry collision sphere radius=0.06602481863; collision sphere radius=0.07959901601
- link iiwa_link_3: geometry collision sphere radius=0.055; collision sphere radius=0.055
- link iiwa_link_4: geometry collision sphere radius=0.06; collision sphere radius=0.06
- link iiwa_link_5: geometry visual mesh filename=package://drake/manipulation/models/iiwa_description/meshes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; visual mesh filename=package://drake/manipulation/models/iiwa_description/meshes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
- link iiwa_link_6: geometry collision sphere radius=0.055; collision sphere radius=0.08
- link iiwa_link_7: geometry collision sphere radius=0.06; visual mesh filename=package://drake/manipulation/models/iiwa_description/meshes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

Commit message: update for move to drake_models

File: manipulation/models/two_link_iiwa14.urdf (robot description, URDF)
Before this commit: robot iiwa14, 10 links, 9 joints
Links:
- link iiwa_link_0: geometry collision cylinder length=0.17 radius=0.139; visual mesh filename=package://drake_models/iiwa_description/meshes/iiwa14/visua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
- link iiwa_link_1: geometry collision sphere radius=0.07959901601; visual mesh filename=package://drake_models/iiwa_description/meshes/iiwa14/visua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
- link iiwa_link_2: geometry collision sphere radius=0.06602481863; collision sphere radius=0.07959901601
- link iiwa_link_3: geometry collision sphere radius=0.055; collision sphere radius=0.055
- link iiwa_link_4: geometry collision sphere radius=0.06; collision sphere radius=0.06
- link iiwa_link_5: geometry visual mesh filename=package://drake_models/iiwa_description/meshes/iiwa14/visua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; visual mesh filename=package://drake_models/iiwa_description/meshes/iiwa14/visua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
- link iiwa_link_6: geometry collision sphere radius=0.055; collision sphere radius=0.08
- link iiwa_link_7: geometry collision sphere radius=0.06; visual mesh filename=package://drake_models/iiwa_description/meshes/iiwa14/visua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
