Commit message: Update Drake to 1.28.0 and update model paths accordingly

File: manipulation/models/pr2_collision_fixed.urdf (robot description, URDF)
Before this commit: robot pr2, 83 links, 83 joints
Links:
- link base_link: geometry collision mesh filename=package://drake_models/pr2_description/meshes/base_v0/base_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; visual mesh filename=package://drake_models/pr2_description/meshes/base_v0/base.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
- link bl_caster_l_wheel_link: geometry visual mesh filename=package://drake_models/pr2_description/meshes/base_v0/wheel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
- link bl_caster_r_wheel_link: geometry visual mesh filename=package://drake_models/pr2_description/meshes/base_v0/wheel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
- link bl_caster_rotation_link: geometry visual mesh filename=package://drake_models/pr2_description/meshes/base_v0/caste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
- link br_caster_l_wheel_link: geometry visual mesh filename=package://drake_models/pr2_description/meshes/base_v0/wheel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
- link br_caster_r_wheel_link: geometry visual mesh filename=package://drake_models/pr2_description/meshes/base_v0/wheel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
- link br_caster_rotation_link: geometry visual mesh filename=package://drake_models/pr2_description/meshes/base_v0/caste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
- link fl_caster_l_wheel_link: geometry visual mesh filename=package://drake_models/pr2_description/meshes/base_v0/wheel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
- link fl_caster_r_wheel_link: geometry visual mesh filename=package://drake_models/pr2_description/meshes/base_v0/wheel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
- link fl_caster_rotation_link: geometry visual mesh filename=package://drake_models/pr2_description/meshes/base_v0/caste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
- link fr_caster_l_wheel_link: geometry visual mesh filename=package://drake_models/pr2_description/meshes/base_v0/wheel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
- link fr_caster_r_wheel_link: geometry visual mesh filename=package://drake_models/pr2_description/meshes/base_v0/wheel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
- link fr_caster_rotation_link: geometry visual mesh filename=package://drake_models/pr2_description/meshes/base_v0/caste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
- link head_pan_link: geometry collision mesh filename=package://drake_models/pr2_description/meshes/head_v0/head_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; visual mesh filename=package://drake_models/pr2_description/meshes/head_v0/head_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
- link head_tilt_link: geometry collision mesh filename=package://drake_models/pr2_description/meshes/head_v0/head_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; visual mesh filename=package://drake_models/pr2_description/meshes/head_v0/head_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
- link l_elbow_flex_link: geometry visual mesh filename=package://drake_models/pr2_description/meshes/upper_arm_v0/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
- link l_forearm_link: geometry collision mesh filename=package://drake_models/pr2_description/meshes/forearm_v0/fo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; visual mesh filename=package://drake_models/pr2_description/meshes/forearm_v0/fo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
- link l_forearm_roll_link: geometry visual mesh filename=package://drake_models/pr2_description/meshes/upper_arm_v0/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
- link l_gripper_l_finger_link: geometry collision mesh filename=package://drake_models/pr2_description/meshes/gripper_v0/l_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; visual mesh filename=package://drake_models/pr2_description/meshes/gripper_v0/l_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
- link l_gripper_l_finger_tip_link: geometry collision mesh filename=package://drake_models/pr2_description/meshes/gripper_v0/l_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; visual mesh filename=package://drake_models/pr2_description/meshes/gripper_v0/l_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
- link l_gripper_palm_link: geometry collision mesh filename=package://drake_models/pr2_description/meshes/gripper_v0/gr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; visual mesh filename=package://drake_models/pr2_description/meshes/gripper_v0/gr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
- link l_gripper_r_finger_link: geometry collision mesh filename=package://drake_models/pr2_description/meshes/gripper_v0/l_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; visual mesh filename=package://drake_models/pr2_description/meshes/gripper_v0/l_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
- link l_gripper_r_finger_tip_link: geometry collision mesh filename=package://drake_models/pr2_description/meshes/gripper_v0/l_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; visual mesh filename=package://drake_models/pr2_description/meshes/gripper_v0/l_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
- link l_shoulder_lift_link: geometry visual mesh filename=package://drake_models/pr2_description/meshes/shoulder_v0/s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
- link l_shoulder_pan_link: geometry collision mesh filename=package://drake_models/pr2_description/meshes/shoulder_v0/s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; visual mesh filename=package://drake_models/pr2_description/meshes/shoulder_v0/s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
- link l_upper_arm_link: geometry collision mesh filename=package://drake_models/pr2_description/meshes/upper_arm_v0/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; visual mesh filename=package://drake_models/pr2_description/meshes/upper_arm_v0/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
- link l_upper_arm_roll_link: geometry visual mesh filename=package://drake_models/pr2_description/meshes/shoulder_v0/u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
- link l_wrist_flex_link: geometry visual mesh filename=package://drake_models/pr2_description/meshes/forearm_v0/wr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
- link l_wrist_roll_link: geometry visual mesh filename=package://drake_models/pr2_description/meshes/forearm_v0/wr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
- link laser_tilt_mount_link: geometry visual mesh filename=package://drake_models/pr2_description/meshes/tilting_laser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
- link r_elbow_flex_link: geometry visual mesh filename=package://drake_models/pr2_description/meshes/upper_arm_v0/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
- link r_forearm_link: geometry collision mesh filename=package://drake_models/pr2_description/meshes/forearm_v0/fo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; visual mesh filename=package://drake_models/pr2_description/meshes/forearm_v0/fo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
- link r_forearm_roll_link: geometry visual mesh filename=package://drake_models/pr2_description/meshes/upper_arm_v0/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
- link r_gripper_l_finger_link: geometry collision mesh filename=package://drake_models/pr2_description/meshes/gripper_v0/l_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; visual mesh filename=package://drake_models/pr2_description/meshes/gripper_v0/l_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
- link r_gripper_l_finger_tip_link: geometry collision mesh filename=package://drake_models/pr2_description/meshes/gripper_v0/l_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; visual mesh filename=package://drake_models/pr2_description/meshes/gripper_v0/l_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
- link r_gripper_palm_link: geometry collision mesh filename=package://drake_models/pr2_description/meshes/gripper_v0/gr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; visual mesh filename=package://drake_models/pr2_description/meshes/gripper_v0/gr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
- link r_gripper_r_finger_link: geometry collision mesh filename=package://drake_models/pr2_description/meshes/gripper_v0/l_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; visual mesh filename=package://drake_models/pr2_description/meshes/gripper_v0/l_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
- link r_gripper_r_finger_tip_link: geometry collision mesh filename=package://drake_models/pr2_description/meshes/gripper_v0/l_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; visual mesh filename=package://drake_models/pr2_description/meshes/gripper_v0/l_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
- link r_shoulder_lift_link: geometry visual mesh filename=package://drake_models/pr2_description/meshes/shoulder_v0/s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
- link r_shoulder_pan_link: geometry collision mesh filename=package://drake_models/pr2_description/meshes/shoulder_v0/s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; visual mesh filename=package://drake_models/pr2_description/meshes/shoulder_v0/s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
- link r_upper_arm_link: geometry collision mesh filename=package://drake_models/pr2_description/meshes/upper_arm_v0/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; visual mesh filename=package://drake_models/pr2_description/meshes/upper_arm_v0/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
- link r_upper_arm_roll_link: geometry visual mesh filename=package://drake_models/pr2_description/meshes/shoulder_v0/u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
- link r_wrist_flex_link: geometry visual mesh filename=package://drake_models/pr2_description/meshes/forearm_v0/wr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
- link r_wrist_roll_link: geometry visual mesh filename=package://drake_models/pr2_description/meshes/forearm_v0/wr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
- link torso_lift_link: geometry collision mesh filename=package://drake_models/pr2_description/meshes/torso_v0/tors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; visual mesh filename=package://drake_models/pr2_description/meshes/torso_v0/tors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
